File: PCB/rtSolder.kicad_pcb (KiCad board)
At the start: 2 copper layers, 81 x 13 mm, 44 parts, among them J1 AudioJack3, J2 Conn_01x05, J3 Jack-DC, Q1 DMP4013LFG-7, SW1 Schurter_1301.9319, SW2 Schurter_1301.9319, U1 LMR14050SDDAR, U2 MIC5233-3.3YS, U3 PIC16F1788-xML, U4 OLED_128x32, U5 TLV333IDCKR

Commit message: adjust temp measurement
changed R19 to 150R
Parts:
- R19: value 110R -> 150R
Changed lines of the file:
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@@
       (effects (font (size 0.5 0.5) (thickness 0.1)) (justify mirror))
     )
-    (fp_text value 110R (at 0 -1.43 90) (layer B.Fab)
+    (fp_text value 150R (at 0 -1.43 90) (layer B.Fab)
       (effects (font (size 1 1) (thickness 0.15)) (justify mirror))
     )

Commit message: last modifications
Connections:
- C1 pad 1: Net-(C1-Pad1) -> (no net)
- C1 pad 2: Net-(C1-Pad2) -> (no net)
- C14 pad 1: Net-(C14-Pad1) -> (no net)
- C9 pad 2: Net-(C9-Pad2) -> (no net)
- D1 pad 1: Net-(C1-Pad1) -> (no net)
- J3 pad 1: Net-(J3-Pad1) -> (no net)
- L1 pad 1: Net-(C1-Pad1) -> (no net)
- Q1 pad 4: Net-(Q1-Pad4) -> (no net)
- Q1 pad 5: Net-(J3-Pad1) -> (no net)
- R1 pad 2: Net-(R1-Pad2) -> (no net)
- R12 pad 1: Net-(Q1-Pad4) -> (no net)
- R15 pad 1: Net-(R15-Pad1) -> (no net)
- R15 pad 2: Net-(R15-Pad2) -> (no net)
- R16 pad 2: Net-(C14-Pad1) -> (no net)
- R17 pad 1: Net-(R15-Pad2) -> (no net)
- R19 pad 1: Net-(R15-Pad1) -> (no net)
- R2 pad 2: Net-(R2-Pad2) -> (no net)
- R20 pad 2: Net-(R20-Pad2) -> (no net)
- R3 pad 2: Net-(R2-Pad2) -> (no net)
- R4 pad 1: Net-(R1-Pad2) -> (no net)
- R5 pad 1: Net-(R2-Pad2) -> (no net)
- R6 pad 2: Net-(R2-Pad2) -> (no net)
- R8 pad 2: Net-(Q1-Pad4) -> (no net)
- U1 pad 1: Net-(C1-Pad2) -> (no net)
- U1 pad 3: Net-(R1-Pad2) -> (no net)
- U1 pad 4: Net-(R20-Pad2) -> (no net)
- U1 pad 5: Net-(R2-Pad2) -> (no net)
- U1 pad 6: Net-(C9-Pad2) -> (no net)
- U1 pad 8: Net-(C1-Pad1) -> (no net)
- U3 pad 11: Net-(U3-Pad11) -> unconnected-(U3-Pad11)
- U3 pad 12: Net-(U3-Pad12) -> unconnected-(U3-Pad12)
- U3 pad 13: Net-(U3-Pad13) -> unconnected-(U3-Pad13)
- U3 pad 14: Net-(U3-Pad14) -> unconnected-(U3-Pad14)
- U3 pad 15: Net-(U3-Pad15) -> unconnected-(U3-Pad15)
- U3 pad 19: Net-(U3-Pad19) -> unconnected-(U3-Pad19)
- U3 pad 20: Net-(U3-Pad20) -> unconnected-(U3-Pad20)
- U3 pad 21: Net-(U3-Pad21) -> unconnected-(U3-Pad21)
- U3 pad 22: Net-(U3-Pad22) -> unconnected-(U3-Pad22)
- U3 pad 23: Net-(U3-Pad23) -> unconnected-(U3-Pad23)
- U3 pad 27: Net-(U3-Pad27) -> unconnected-(U3-Pad27)
- U3 pad 28: Net-(U3-Pad28) -> unconnected-(U3-Pad28)
- U3 pad 3: Net-(U3-Pad3) -> unconnected-(U3-Pad3)
- U3 pad 4: Net-(U3-Pad4) -> unconnected-(U3-Pad4)
- U3 pad 6: Net-(U3-Pad6) -> unconnected-(U3-Pad6)
- U4 pad 3: Net-(U3-Pad11) -> unconnected-(U3-Pad11)
- U4 pad 4: Net-(U3-Pad12) -> unconnected-(U3-Pad12)
- U5 pad 1: Net-(C14-Pad1) -> (no net)
- U5 pad 3: Net-(R15-Pad1) -> (no net)
- U5 pad 4: Net-(R15-Pad2) -> (no net)
Routing:
- net (no net): track 0.00 -> 102.2 mm, vias 0 -> 13
- net Net-(R2-Pad2): track 51.7 -> 0.00 mm, vias 3 -> 0
- net Net-(U3-Pad11): track 35.0 -> 0.00 mm, vias 1 -> 0
- net unconnected-(U3-Pad11): track 0.00 -> 35.0 mm, vias 0 -> 1
- net unconnected-(U3-Pad12): track 0.00 -> 31.1 mm, vias 0 -> 1
- net Net-(U3-Pad12): track 31.1 -> 0.00 mm, vias 1 -> 0
- net Net-(C14-Pad1): track 10.9 -> 0.00 mm, vias 2 -> 0
- net Net-(C1-Pad1): track 10.4 -> 0.00 mm, vias 6 -> 0
- net Net-(R1-Pad2): track 9.46 -> 0.00 mm
- net Net-(R15-Pad2): track 6.15 -> 0.00 mm, vias 2 -> 0
- net Net-(Q1-Pad4): track 4.13 -> 0.00 mm
- net Net-(R15-Pad1): track 3.11 -> 0.00 mm
- net Net-(C9-Pad2): track 2.19 -> 0.00 mm
- net Net-(C1-Pad2): track 2.09 -> 0.00 mm
- net Net-(R20-Pad2): track 2.08 -> 0.00 mm
- added copper zone on B.Cu, net (none)
- added copper zone on F.Cu, net (none)
- removed copper zone on B.Cu, net Net-(C1-Pad1)
- removed copper zone on F.Cu, net Net-(C1-Pad1)
- removed copper zone on B.Cu, net Net-(J3-Pad1)
Other:
- net class Default removed
